Commit message: updating to have d435 in Gazebo

File: ros_ws/src/maxwell_gazebo/urdf/maxwell_swerve.urdf (robot description, URDF)
Before this commit: robot maxwell_rover, 11 links, 10 joints
Links:
- added link camera_color_frame
- added link camera_color_optical_frame
- added link camera_depth_frame
- added link camera_depth_optical_frame
Joints:
- added joint camera_color_joint: type fixed, parent Camera_link, child camera_color_frame, origin xyz=0 0 0 rpy=0 0 0
- added joint camera_color_optical_joint: type fixed, parent camera_color_frame, child camera_color_optical_frame, origin xyz=0 0 0 rpy=-1.5708 0 -1.5708
- added joint camera_depth_joint: type fixed, parent Camera_link, child camera_depth_frame, origin xyz=0 0 0 rpy=0 0 0
- added joint camera_depth_optical_joint: type fixed, parent camera_depth_frame, child camera_depth_optical_frame, origin xyz=0 0 0 rpy=-1.5708 0 -1.5708

Commit message: Full URDF from Conversion

File: ros_ws/src/maxwell_gazebo/urdf/maxwell_swerve.urdf (robot description, URDF)
Before this commit: robot maxwell_rover, 15 links, 14 joints
Links:
- link BL_Link: geometry collision cylinder length=0.1 radius=0.127; visual mesh filename=package://maxwell_description/meshes/BL_Link.STL
- link BR_Link: geometry collision cylinder length=0.1 radius=0.127; visual mesh filename=package://maxwell_description/meshes/BR_Link.STL
- link Base_link: geometry collision box size=0.8 0.6 0.3; visual mesh filename=package://maxwell_description/meshes/Base_link.STL
- link FL_Link: geometry collision cylinder length=0.1 radius=0.127; visual mesh filename=package://maxwell_description/meshes/FL_Link.STL
- link FR_Link: geometry collision cylinder length=0.1 radius=0.127; visual mesh filename=package://maxwell_description/meshes/FR_Link.STL

Commit message: Adding IMU at the camera of the rover

File: ros_ws/src/maxwell_gazebo/urdf/maxwell_swerve.urdf (robot description, URDF)
Before this commit: robot maxwell_rover, 15 links, 14 joints
Links:
- added link camera_imu_link, mass 0.01
Joints:
- added joint camera_imu_joint: type fixed, parent Camera_link, child camera_imu_link, origin xyz=0 0 0 rpy=0 0 0
