Commit message: small changes to packages and updating urdfs in description folder

File: ros_ws/src/maxwell_description/urdf/PROPER_Simplified Rover.SLDASM.urdf (robot description, URDF)
Before this commit: robot PROPER_Simplified Rover.SLDASM, 10 links, 9 joints
Links:
- link BL_Link: geometry collision mesh filename=/home/koener/Documents/MMRT_2025_Autonomy/ros2_ws/src/maxwe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; visual mesh filename=/home/koener/Documents/MMRT_2025_Autonomy/ros2_ws/src/maxwe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
- link BL_Rot_Link: geometry collision mesh filename=/home/koener/Documents/MMRT_2025_Autonomy/ros2_ws/src/maxwe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; visual mesh filename=/home/koener/Documents/MMRT_2025_Autonomy/ros2_ws/src/maxwe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
- link BR_Link: geometry collision mesh filename=/home/koener/Documents/MMRT_2025_Autonomy/ros2_ws/src/maxwe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; visual mesh filename=/home/koener/Documents/MMRT_2025_Autonomy/ros2_ws/src/maxwe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
- link BR_Rot_Link: geometry collision mesh filename=/home/koener/Documents/MMRT_2025_Autonomy/ros2_ws/src/maxwe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; visual mesh filename=/home/koener/Documents/MMRT_2025_Autonomy/ros2_ws/src/maxwe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
- link Base_link: geometry collision mesh filename=/home/koener/Documents/MMRT_2025_Autonomy/ros2_ws/src/maxwe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; visual mesh filename=/home/koener/Documents/MMRT_2025_Autonomy/ros2_ws/src/maxwe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
- link Camera_link: geometry collision mesh filename=/home/koener/Documents/MMRT_2025_Autonomy/ros2_ws/src/maxwe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; visual mesh filename=/home/koener/Documents/MMRT_2025_Autonomy/ros2_ws/src/maxwe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
- link FL_Link: geometry collision mesh filename=/home/koener/Documents/MMRT_2025_Autonomy/ros2_ws/src/maxwe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; visual mesh filename=/home/koener/Documents/MMRT_2025_Autonomy/ros2_ws/src/maxwe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
- link FL_Rot_Link: geometry collision mesh filename=/home/koener/Documents/MMRT_2025_Autonomy/ros2_ws/src/maxwe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; visual mesh filename=/home/koener/Documents/MMRT_2025_Autonomy/ros2_ws/src/maxwe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
- link FR_Link: geometry collision mesh filename=/home/koener/Documents/MMRT_2025_Autonomy/ros2_ws/src/maxwe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; visual mesh filename=/home/koener/Documents/MMRT_2025_Autonomy/ros2_ws/src/maxwe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
- link FR_Rot_Link: geometry collision mesh filename=/home/koener/Documents/MMRT_2025_Autonomy/ros2_ws/src/maxwe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; visual mesh filename=/home/koener/Documents/MMRT_2025_Autonomy/ros2_ws/src/maxwe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
